Commit message: assets: update robot model to URDF V4

File: assets/sh_dog/raw/urdf/URDF-V4-test1.urdf (robot description, URDF)
Before this commit: robot urdf-v2-2, 17 links, 16 joints
Links:
- link base_link: mass 5.7993 -> 6.9493; geometry collision mesh filename=package://URDF-V4-test1/meshes/base_link.STL; visual mesh filename=package://URDF-V4-test1/meshes/base_link.STL
- link fl_abad_link: geometry collision mesh filename=package://URDF-V4-test1/meshes/fl_abad_link.STL; visual mesh filename=package://URDF-V4-test1/meshes/fl_abad_link.STL
- link fl_foot_link: geometry collision mesh filename=package://URDF-V4-test1/meshes/fl_foot_link.STL; visual mesh filename=package://URDF-V4-test1/meshes/fl_foot_link.STL
- link fl_hip_link: mass 1.25750624804615 -> 1.2575; geometry collision mesh filename=package://URDF-V4-test1/meshes/fl_hip_link.STL; visual mesh filename=package://URDF-V4-test1/meshes/fl_hip_link.STL
- link fl_knee_link: geometry collision mesh filename=package://URDF-V4-test1/meshes/fl_knee_link.STL; visual mesh filename=package://URDF-V4-test1/meshes/fl_knee_link.STL
- link fr_abad_link: mass 0.928856365893587 -> 0.92886; geometry collision mesh filename=package://URDF-V4-test1/meshes/fr_abad_link.STL; visual mesh filename=package://URDF-V4-test1/meshes/fr_abad_link.STL
- link fr_foot_link: geometry collision mesh filename=package://URDF-V4-test1/meshes/fr_foot_link.STL; visual mesh filename=package://URDF-V4-test1/meshes/fr_foot_link.STL
- link fr_hip_link: mass 1.25749406115706 -> 1.25749406115707; geometry collision mesh filename=package://URDF-V4-test1/meshes/fr_hip_link.STL; visual mesh filename=package://URDF-V4-test1/meshes/fr_hip_link.STL
- link fr_knee_link: geometry collision mesh filename=package://URDF-V4-test1/meshes/fr_knee_link.STL; visual mesh filename=package://URDF-V4-test1/meshes/fr_knee_link.STL
- link rl_abad_link: geometry collision mesh filename=package://URDF-V4-test1/meshes/rl_abad_link.STL; visual mesh filename=package://URDF-V4-test1/meshes/rl_abad_link.STL
- link rl_foot_link: geometry collision mesh filename=package://URDF-V4-test1/meshes/rl_foot_link.STL; visual mesh filename=package://URDF-V4-test1/meshes/rl_foot_link.STL
- link rl_hip_link: geometry collision mesh filename=package://URDF-V4-test1/meshes/rl_hip_link.STL; visual mesh filename=package://URDF-V4-test1/meshes/rl_hip_link.STL
- link rl_knee_link: geometry collision mesh filename=package://URDF-V4-test1/meshes/rl_knee_link.STL; visual mesh filename=package://URDF-V4-test1/meshes/rl_knee_link.STL
- link rr_abad_link: geometry collision mesh filename=package://URDF-V4-test1/meshes/rr_abad_link.STL; visual mesh filename=package://URDF-V4-test1/meshes/rr_abad_link.STL
- link rr_foot_link: geometry collision mesh filename=package://URDF-V4-test1/meshes/rr_foot_link.STL; visual mesh filename=package://URDF-V4-test1/meshes/rr_foot_link.STL
- link rr_hip_link: geometry collision mesh filename=package://URDF-V4-test1/meshes/rr_hip_link.STL; visual mesh filename=package://URDF-V4-test1/meshes/rr_hip_link.STL
- link rr_knee_link: geometry collision mesh filename=package://URDF-V4-test1/meshes/rr_knee_link.STL; visual mesh filename=package://URDF-V4-test1/meshes/rr_knee_link.STL
Joints:
- joint fr_foot_joint: origin xyz=0.0219999999999999 0 -0.225 rpy=0 0 0 -> xyz=0.022 0 -0.225 rpy=0 0 0

File: assets/sh_dog/urdf/sh_dog.urdf (robot description, URDF)
Before this commit: robot sh_dog, 17 links, 16 joints
Links:
- link base_link: mass 5.7993 -> 6.9493
- link fl_hip_link: mass 1.25750624804615 -> 1.2575
- link fr_abad_link: mass 0.928856365893587 -> 0.92886
- link fr_hip_link: mass 1.25749406115706 -> 1.25749406115707
Joints:
- joint fr_foot_joint: origin xyz=0.0219999999999999 0 -0.225 rpy=0 0 0 -> xyz=0.022 0 -0.225 rpy=0 0 0
