Commit message: assets: define primitive collision model

File: assets/sh_dog/urdf/sh_dog.urdf (robot description, URDF)
Before this commit: robot sh_dog, 17 links, 16 joints
Links:
- link base_link: geometry collision box size=0.29 0.142 0.13; visual mesh filename=../raw/meshes/base_link.STL
- link fl_abad_link: geometry collision cylinder length=0.08 radius=0.046; visual mesh filename=../raw/meshes/fl_abad_link.STL
- link fl_foot_link: geometry collision sphere radius=0.0225; visual mesh filename=../raw/meshes/fl_foot_link.STL
- link fl_hip_link: geometry collision box size=0.065 0.04 0.11; visual mesh filename=../raw/meshes/fl_hip_link.STL
- link fl_knee_link: geometry collision cylinder length=0.14 radius=0.015; visual mesh filename=../raw/meshes/fl_knee_link.STL
- link fr_abad_link: geometry collision cylinder length=0.08 radius=0.046; visual mesh filename=../raw/meshes/fr_abad_link.STL
- link fr_foot_link: geometry collision sphere radius=0.0225; visual mesh filename=../raw/meshes/fr_foot_link.STL
- link fr_hip_link: geometry collision box size=0.065 0.04 0.11; visual mesh filename=../raw/meshes/fr_hip_link.STL
- link fr_knee_link: geometry collision cylinder length=0.14 radius=0.015; visual mesh filename=../raw/meshes/fr_knee_link.STL
- link rl_abad_link: geometry collision cylinder length=0.08 radius=0.046; visual mesh filename=../raw/meshes/rl_abad_link.STL
- link rl_foot_link: geometry collision sphere radius=0.0225; visual mesh filename=../raw/meshes/rl_foot_link.STL
- link rl_hip_link: geometry collision box size=0.065 0.04 0.11; visual mesh filename=../raw/meshes/rl_hip_link.STL
- link rl_knee_link: geometry collision cylinder length=0.14 radius=0.015; visual mesh filename=../raw/meshes/rl_knee_link.STL
- link rr_abad_link: geometry collision cylinder length=0.08 radius=0.046; visual mesh filename=../raw/meshes/rr_abad_link.STL
- link rr_foot_link: geometry collision sphere radius=0.0225; visual mesh filename=../raw/meshes/rr_foot_link.STL
- link rr_hip_link: geometry collision box size=0.065 0.04 0.11; visual mesh filename=../raw/meshes/rr_hip_link.STL
- link rr_knee_link: geometry collision cylinder length=0.14 radius=0.015; visual mesh filename=../raw/meshes/rr_knee_link.STL

Commit message: assets: add compound primitive collisions

File: assets/sh_dog/urdf/sh_dog.urdf (robot description, URDF)
Before this commit: robot sh_dog, 17 links, 16 joints
Links:
- link base_link: geometry collision box size=0.09 0.19 0.1; collision box size=0.09 0.19 0.1
- link fl_abad_link: geometry collision cylinder length=0.06 radius=0.041; collision cylinder length=0.08 radius=0.046
- link fl_hip_link: geometry collision box size=0.07 0.034 0.18; collision cylinder length=0.09 radius=0.04
- link fl_knee_link: geometry collision cylinder length=0.13 radius=0.014; collision cylinder length=0.15 radius=0.018
- link fr_abad_link: geometry collision cylinder length=0.06 radius=0.041; collision cylinder length=0.08 radius=0.046
- link fr_hip_link: geometry collision box size=0.07 0.034 0.18; collision cylinder length=0.09 radius=0.04
- link fr_knee_link: geometry collision cylinder length=0.13 radius=0.014; collision cylinder length=0.15 radius=0.018
- link rl_abad_link: geometry collision cylinder length=0.06 radius=0.041; collision cylinder length=0.08 radius=0.046
- link rl_hip_link: geometry collision box size=0.07 0.034 0.18; collision cylinder length=0.09 radius=0.04
- link rl_knee_link: geometry collision cylinder length=0.13 radius=0.014; collision cylinder length=0.15 radius=0.018
- link rr_abad_link: geometry collision cylinder length=0.06 radius=0.041; collision cylinder length=0.08 radius=0.046
- link rr_hip_link: geometry collision box size=0.07 0.034 0.18; collision cylinder length=0.09 radius=0.04
- link rr_knee_link: geometry collision cylinder length=0.13 radius=0.014; collision cylinder length=0.15 radius=0.018
